File: esp-master kicad/esp-master-nodeMCU/esp-master-nodeMCU.kicad_sch (KiCad schematic)
At the start: 20 parts, among them J1 Conn_01x06_Female, J2 Conn_01x06_Male, J3 Conn_01x06_Female, J4 Conn_01x06_Male, J5 Conn_01x07_Male, J6 Conn_01x07_Female, J7 SD_Card, J8 Conn_01x06_Female, J9 Conn_01x06_Male, SW1 SW_Push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

Commit message: Update esp-master-nodeMCU.kicad_sch
Parts:
- C1: value C_Polarized -> 2200uF
- C2: value C -> 33pF
- C3: value C -> 10pF
Changed lines of the file:
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@@
       (effects (font (size 1.27 1.27)) (justify left))
     )
-    (property "Value" "C" (id 1) (at 146.05 38.1 0)
+    (property "Value" "33pF" (id 1) (at 146.05 38.1 0)
       (effects (font (size 1.27 1.27)) (justify left))
     )
@@
       (effects (font (size 1.27 1.27)) (justify left))
     )
-    (property "Value" "C_Polarized" (id 1) (at 125.73 38.1 0)
+    (property "Value" "2200uF" (id 1) (at 125.73 38.1 0)
       (effects (font (size 1.27 1.27)) (justify left))
     )
@@
       (effects (font (size 1.27 1.27)) (justify left))
     )
-    (property "Value" "C" (id 1) (at 158.75 38.1 0)
+    (property "Value" "10pF" (id 1) (at 158.75 38.1 0)
       (effects (font (size 1.27 1.27)) (justify left))
     )
@@
     )
     (path "/37551ef5-1a93-4655-9635-abdd4742c8aa"
-      (reference "C1") (unit 1) (value "C_Polarized") (footprint "")
+      (reference "C1") (unit 1) (value "2200uF") (footprint "")
     )
     (path "/09b4820b-cacf-4ab6-bc1c-27905b41c380"
-      (reference "C2") (unit 1) (value "C") (footprint "")
+      (reference "C2") (unit 1) (value "33pF") (footprint "")
     )
     (path "/53675dc1-84df-46b5-8cc9-715e2017b317"
-      (reference "C3") (unit 1) (value "C") (footprint "")
+      (reference "C3") (unit 1) (value "10pF") (footprint "")
     )
     (path "/c2bbfd57-799e-45c5-b16f-899657985044"
