File: esp-merged kicad/esp-merged_v1/esp-merged_v1.kicad_sch (KiCad schematic)
At the start: 15 parts

Commit message: postępy projektowania PCB
Parts:
- added C?: 100nF, Capacitor_Tantalum_SMD:CP_EIA-1608-08_AVX-J_Pad1.25x1.05mm_HandSolder, symbol Device:C
- added J?: Conn_02x04_Male, wlasne_footprinty:prog pins ESP32 (aka esp01), symbol Connector:Conn_01x08_Male
- added R: 10K, symbol Device:R
- added SW?: SW_Push, symbol Switch:SW_Push
- J?: footprint (none) -> wlasne_footprinty:screw connector 12
- S?: footprint (none) -> wlasne_footprinty:MH-sensor-series
Connections:
- net 3.3 VCC: now also J?.1 (Pin_1), R.1
- net GND: now also C?.1, J?.8 (Pin_8), SW?.1
- net PROG_I0: now reaches U?.25 (IO0)
- net PROG_I0: now also J?.2 (Pin_2)
- net PROG_EN: now reaches U?.3 (EN)
- net PROG_EN: now also C?.2, J?.3 (Pin_3), R.2, SW?.2
- net PROG_TX: now reaches U?.34 (RXD0/IO3)
- net PROG_TX: now also J?.4 (Pin_4)
- net PROG_RX: now reaches U?.35 (TXD0/IO1)
- net PROG_RX: now also J?.5 (Pin_5)
- no-connect marks 16 -> 19
Other:
- note added: "Wyjścia do programowania w układzie esp-01, tak aby możliwe było połączenie poprzez programator (umieścić na zewnątrz płytki w tym celu, a piny męskie dłuższą stroną na dół)"
- note added: "pamiętać, że pcb ma być SLIM (cienkie), czyli wszystko będzie kładzione bokiem"
- note added: "todo footprint: baterii SIM800L HX711 karty sd"
- note removed: "TODO piny out do programowania esp (przyciski en i reset oraz tx/rx)"

Commit message: postepy kicad, footprinty
Parts:
- BT?: footprint (none) -> wlasne_footprinty:koszyk na baterie 1x1
- J?: footprint (none) -> wlasne_footprinty:karta sd
- M?: footprint (none) -> wlasne_footprinty:hx711
- U?: footprint Package_SO:SOIC-16W_7.5x10.3mm_P1.27mm -> wlasne_footprinty:ds3231
Other:
- note added: "todo footprint: SIM800L"
- note added: "todo jako antene dać wyjście odpowiednie do podłączenia PCB pod kabel i kablem do anteny"
- note removed: "todo footprint: baterii SIM800L HX711 karty sd"
Changed lines of the file:
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@@
     (effects (font (size 1.27 1.27)) (justify left bottom))
   )
-  (text "todo\nfootprint:\n	baterii\n	SIM800L\n	HX711\n	karty sd"
-    (at 93.345 157.48 0)
+  (text "todo\nfootprint:\n	SIM800L" (at 93.345 157.48 0)
     (effects (font (size 1.27 1.27)) (justify left bottom))
   )
   (text "Zegar czasu rzeczywistego" (at 158.75 31.115 0)
+    (effects (font (size 1.27 1.27)) (justify left bottom))
+  )
+  (text "todo jako antene dać wyjście odpowiednie do podłączenia PCB pod kabel i kablem do anteny "
+    (at 56.515 184.785 0)
     (effects (font (size 1.27 1.27)) (justify left bottom))
   )
@@
     (property "Reference" "J?" (id 0) (at 270.51 59.055 0))
     (property "Value" "SD_Card" (id 1) (at 273.05 56.515 0))
-    (property "Footprint" "" (id 2) (at 247.65 45.085 0)
+    (property "Footprint" "wlasne_footprinty:karta sd" (id 2) (at 247.65 45.085 0)
       (effects (font (size 1.27 1.27)) hide)
     )
@@
     (property "Reference" "M?" (id 0) (at 213.995 70.485 0))
     (property "Value" "HX711" (id 1) (at 213.995 73.025 0))
-    (property "Footprint" "" (id 2) (at 215.9 92.075 0)
+    (property "Footprint" "wlasne_footprinty:hx711" (id 2) (at 215.9 92.075 0)
       (effects (font (size 1.27 1.27)) hide)
     )
@@
       (effects (font (size 1.27 1.27)) (justify left))
     )
-    (property "Footprint" "Package_SO:SOIC-16W_7.5x10.3mm_P1.27mm" (id 2) (at 181.61 62.865 0)
+    (property "Footprint" "wlasne_footprinty:ds3231" (id 2) (at 181.61 62.865 0)
       (effects (font (size 1.27 1.27)) hide)
     )
@@
       (effects (font (size 1.27 1.27)) (justify left))
     )
-    (property "Footprint" "" (id 2) (at 17.78 49.911 90)
+    (property "Footprint" "wlasne_footprinty:koszyk na baterie 1x1" (id 2) (at 17.78 49.911 90)
       (effects (font (size 1.27 1.27)) hide)
     )
@@
     )
     (path "/fdae1537-0230-405c-818b-09f62494491f"
-      (reference "BT?") (unit 1) (value "Battery") (footprint "")
+      (reference "BT?") (unit 1) (value "Battery") (footprint "wlasne_footprinty:koszyk na baterie 1x1")
     )
     (path "/543b574d-f4f4-4981-80a0-26a8cf3efc80"
@@
     )
     (path "/15aa75da-45cd-42cf-9e21-383f7cc14908"
-      (reference "J?") (unit 1) (value "SD_Card") (footprint "")
+      (reference "J?") (unit 1) (value "SD_Card") (footprint "wlasne_footprinty:karta sd")
     )
     (path "/2f60fd02-4c6d-4755-a6da-591f500d5fc2"
@@
     )
     (path "/3e906b60-a74c-43dd-bad1-f706f0b88384"
-      (reference "M?") (unit 1) (value "HX711") (footprint "")
+      (reference "M?") (unit 1) (value "HX711") (footprint "wlasne_footprinty:hx711")
     )
     (path "/f942f231-666a-422f-9054-604298697935"
@@
     )
     (path "/846ab384-d5c4-4270-84d2-d920f019659c"
-      (reference "U?") (unit 1) (value "DS3231M") (footprint "Package_SO:SOIC-16W_7.5x10.3mm_P1.27mm")
+      (reference "U?") (unit 1) (value "DS3231M") (footprint "wlasne_footprinty:ds3231")
     )
     (path "/d61b37e6-1acd-4826-b1f1-a50ad37b0751"

Commit message: kicad footprint sim800l
Parts:
- U?: footprint (none) -> wlasne_footprinty:sim800l
Other:
- note added: "todo footprint: diody, rezystory, konden"
- note removed: "todo footprint: SIM800L"
Changed lines of the file:
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@@
     (effects (font (size 1.27 1.27)) (justify left bottom))
   )
-  (text "todo\nfootprint:\n	SIM800L" (at 93.345 157.48 0)
+  (text "todo\nfootprint:\n	diody, rezystory, konden" (at 93.345 157.48 0)
     (effects (font (size 1.27 1.27)) (justify left bottom))
   )
@@
     (property "Reference" "U?" (id 0) (at 143.51 123.19 0))
     (property "Value" "SIM800L" (id 1) (at 143.51 125.73 0))
-    (property "Footprint" "" (id 2) (at 144.78 99.695 0)
+    (property "Footprint" "wlasne_footprinty:sim800l" (id 2) (at 144.78 99.695 0)
       (effects (font (size 1.27 1.27)) hide)
     )
@@
       (effects (font (size 1.27 1.27)) hide)
     )
-    (pin "")
     (pin "0")
     (pin "1")
     (pin "10")
+    (pin "11")
     (pin "2")
     (pin "3")
@@
     )
     (path "/db9994ff-c050-4c43-8a3d-c4f5d72639c2"
-      (reference "U?") (unit 1) (value "SIM800L") (footprint "")
-    )
-  )
+      (reference "U?") (unit 1) (value "SIM800L") (footprint "wlasne_footprinty:sim800l")
+    )
+  )

Commit message: pcb skonczone?
Parts:
- AE1: renamed from AE?; footprint (none) -> Connector_Coaxial:SMA_Amphenol_132291_Vertical; opis (none) -> SMA
- C1: renamed from C?; footprint Capacitor_Tantalum_SMD:CP_EIA-1608-08_AVX-J_Pad1.25x1.05mm_HandSolder -> Capacitor_THT:CP_Radial_Tantal_D5.0mm_P2.50mm
- C2: renamed from C?; footprint (none) -> Capacitor_THT:CP_Radial_D10.0mm_P5.00mm
- C3, C4: renamed from C?; footprint (none) -> Capacitor_THT:CP_Radial_Tantal_D5.0mm_P2.50mm
- D1: renamed from D?; footprint (none) -> Diode_THT:D_A-405_P10.16mm_Horizontal
- F1: renamed from F?; footprint (none) -> Resistor_THT:R_Axial_DIN0411_L9.9mm_D3.6mm_P15.24mm_Horizontal
- J1: renamed from J?; footprint wlasne_footprinty:prog pins ESP32 (aka esp01) -> wlasne_footprinty:prog pins ESP32 (aka esp01) v2 (odwrocone)
- R1: renamed from R; footprint (none) -> Resistor_THT:R_Axial_DIN0207_L6.3mm_D2.5mm_P10.16mm_Horizontal
- SW1: renamed from SW?; footprint (none) -> wlasne_footprinty:wlacznik
- SW2: renamed from SW?; footprint (none) -> wlasne_footprinty:mały button
- gave numbers to parts that had none: 8
Connections:
- net 3.3 VCC: now also D1.1 (A); no longer D1.2 (A)
- net Battery VCC: now also D1.2 (K), F1.2; no longer BT1.1 (+), SW1.1
- net GND: no longer U3.10 (GND), U3.11 (GND), U3.12 (GND), U3.5 (GND), U3.6 (GND), U3.7 (GND), U3.8 (GND), U3.9 (GND)
- new net: BT1.1 (+), SW1.1
- no-connect marks 19 -> 36
Other:
- note added: "Wyjścia do programowania w układzie esp-01, tak aby możliwe było połączenie poprzez programator (męskie piny do góry płytki, elementem odwracanym jest adapter)"
- note added: "todo rozważyć orientację i stronę po której będzie footprint do interfrejsu PROG, jeśli się okaże że wszystkie komponenty będą po jednej stronie to możliwe, że żeby programować płytkę będzie trzeba ją do góry nogami dać do adaptera, więc obecny footprint może musieć być na odwrót"
- note added: "todo sw1 to jest inny przycisk, ten przełączany todo footprint"
- note removed: "Wyjścia do programowania w układzie esp-01, tak aby możliwe było połączenie poprzez programator (umieścić na zewnątrz płytki w tym celu, a piny męskie dłuższą stroną na dół)"
- note removed: "pamiętać, że pcb ma być SLIM (cienkie), czyli wszystko będzie kładzione bokiem"
- note removed: "todo footprint: diody, rezystory, konden"
