File: esp-merged kicad/esp-merged_v2/esp-merged_v2.kicad_pcb (KiCad board)
At the start: 2 copper layers, 100 x 100 mm, 19 parts, among them J1 Conn_02x04_Male, J2 SD_Card, J3 Screw_Terminal_01x12, M1 HX711, SW1 SW_Push, SW2 SW_Push, U1 ESP32-WROOM-32, U2 SIM800L, U3 DS3231M

Commit message: a
Changed lines of the file:
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@@
       (usegerberattributes true)
       (usegerberadvancedattributes true)
-      (creategerberjobfile true)
+      (creategerberjobfile false)
       (svguseinch false)
       (svgprecision 6)
@@
       (outputformat 1)
       (mirror false)
-      (drillshape 1)
+      (drillshape 0)
       (scaleselection 1)
       (outputdirectory "")
@@
     (property "Sheetname" "")
     (attr through_hole)
-    (fp_text reference "BT1" (at 7.874 24.892 -90 unlocked) (layer "F.SilkS")
+    (fp_text reference "BT1" (at 12.666 13.535 unlocked) (layer "F.SilkS")
       (effects (font (size 1 1) (thickness 0.15)))
     )
@@
     (property "Sheetname" "")
     (attr through_hole)
-    (fp_text reference "U2" (at 0 -0.5 180 unlocked) (layer "F.SilkS")
+    (fp_text reference "U2" (at 12.905 11.655 unlocked) (layer "F.SilkS")
       (effects (font (size 1 1) (thickness 0.15)))
     )
@@
     (property "Sheetname" "")
     (attr through_hole)
-    (fp_text reference "D1" (at 5.08 2.5 90) (layer "F.SilkS")
+    (fp_text reference "D1" (at 5.08 -2.6 90) (layer "F.SilkS")
       (effects (font (size 1 1) (thickness 0.15)))
     )
     (fp_text value "DIODE" (at 5.58 -2.5 90) (layer "F.Fab")
-      (effects (font (size 1 1) (thickness 0.15)))
-    )
-    (fp_text user "K" (at 0 -1.9 90) (layer "F.SilkS")
       (effects (font (size 1 1) (thickness 0.15)))
     )
@@
     (property "Sheetname" "")
     (attr through_hole)
-    (fp_text reference "J2" (at 19.558 11.176 180 unlocked) (layer "F.SilkS")
+    (fp_text reference "J2" (at 1.855 1.735 unlocked) (layer "F.SilkS")
       (effects (font (size 1 1) (thickness 0.15)))
     )
@@
     (property "Sheetname" "")
     (attr through_hole)
-    (fp_text reference "F1" (at 7.62 -2.92 90) (layer "F.SilkS")
+    (fp_text reference "F1" (at 7.62 3.1 90) (layer "F.SilkS")
       (effects (font (size 1 1) (thickness 0.15)))
     )
@@
     (property "Sheetname" "")
     (attr through_hole)
-    (fp_text reference "R1" (at 5.08 2.5) (layer "F.SilkS")
+    (fp_text reference "R1" (at 4.88 -2.4) (layer "F.SilkS")
       (effects (font (size 1 1) (thickness 0.15)))
     )
@@
     (property "Sheetname" "")
     (attr through_hole)
-    (fp_text reference "SW1" (at 1.055 -1.38 unlocked) (layer "F.SilkS")
+    (fp_text reference "SW1" (at 14.055 -1.58 unlocked) (layer "F.SilkS")
       (effects (font (size 1 1) (thickness 0.15)))
     )
@@
     (property "opis" "LOW ESR")
     (attr through_hole)
-    (fp_text reference "C2" (at 2.5 -6.25 90) (layer "F.SilkS")
+    (fp_text reference "C2" (at -2.932323 3 180) (layer "F.SilkS")
       (effects (font (size 1 1) (thickness 0.15)))
     )
@@
     (property "Sheetname" "")
     (attr through_hole)
-    (fp_text reference "J3" (at 0 -0.5 90 unlocked) (layer "F.SilkS")
+    (fp_text reference "J3" (at -1.055 2.955 unlocked) (layer "F.SilkS")
       (effects (font (size 1 1) (thickness 0.15)))
     )
@@
     (property "Sheetname" "")
     (attr through_hole)
-    (fp_text reference "S1" (at 14.224 4.826 unlocked) (layer "F.SilkS")
+    (fp_text reference "S1" (at 15.955 6.805 unlocked) (layer "F.SilkS")
       (effects (font (size 1 1) (thickness 0.15)))
     )
@@
     (property "Sheetname" "")
     (attr through_hole)
-    (fp_text reference "M1" (at 16.51 10.16 90 unlocked) (layer "F.SilkS")
+    (fp_text reference "M1" (at 16.51 10.255 unlocked) (layer "F.SilkS")
       (effects (font (size 1 1) (thickness 0.15)))
     )
@@
     (property "Sheetname" "")
     (attr smd)
-    (fp_text reference "U1" (at -10.61 8.43 90) (layer "F.SilkS")
+    (fp_text reference "U1" (at -0.3 4.4 180) (layer "F.SilkS")
       (effects (font (size 1 1) (thickness 0.15)))
     )
@@
     (property "Sheetname" "")
     (attr through_hole)
-    (fp_text reference "SW2" (at 3.455 6.955 unlocked) (layer "F.SilkS")
+    (fp_text reference "SW2" (at 2.955 7.2 unlocked) (layer "F.SilkS")
       (effects (font (size 1 1) (thickness 0.15)))
     )
@@
     (property "Sheetname" "")
     (attr through_hole)
-    (fp_text reference "U3" (at 19.558 10.16 -90 unlocked) (layer "F.SilkS")
+    (fp_text reference "U3" (at 19.38 10.205 unlocked) (layer "F.SilkS")
       (effects (font (size 1 1) (thickness 0.15)))
     )
@@
     (property "Sheetname" "")
     (attr through_hole)
-    (fp_text reference "C1" (at -2.294888 0 90) (layer "F.SilkS")
+    (fp_text reference "C1" (at 1.005112 -3.7 180) (layer "F.SilkS")
       (effects (font (size 1 1) (thickness 0.15)))
     )
@@
       (effects (font (size 1 1) (thickness 0.15)))
     )
-    (fp_text user "PROG" (at -5.818 0.803 90 unlocked) (layer "F.SilkS")
+    (fp_text user "PROG" (at -9.769 10.555 unlocked) (layer "F.SilkS")
       (effects (font (size 1 1) (thickness 0.15)))
     )
@@
       (net 3 "GND") (pinfunction "Pin_8") (pintype "passive"))
   )
-  (gr_circle (center 254 34.5) (end 257 34.5) (layer "F.SilkS") (width 0.1) (fill none))
-  (gr_circle (center 254 131.45) (end 257 131.45) (layer "F.SilkS") (width 0.1) (fill none))
-  (gr_circle (center 164.95 131.45) (end 167.95 131.45) (layer "F.SilkS") (width 0.1) (fill none))
-  (gr_circle (center 164.95 34.5) (end 167.95 34.5) (layer "F.SilkS") (width 0.1) (fill none))
+  (gr_circle (center 254 34.5) (end 254.8 34.4) (layer "F.SilkS") (width 0.1) (fill none))
+  (gr_circle (center 254 131.45) (end 255 131.2) (layer "F.SilkS") (width 0.1) (fill none))
+  (gr_circle (center 164.95 131.45) (end 166 131.2) (layer "F.SilkS") (width 0.1) (fill none))
+  (gr_circle (center 164.95 34.5) (end 165.9 34.5) (layer "F.SilkS") (width 0.1) (fill none))
   (gr_rect (start 159 133.2) (end 259 33.2) (layer "Edge.Cuts") (width 0.1) (fill none))
-  (gr_text "JLCJLCJLCJLC" (at 170 82.3 270) (layer "F.SilkS")
+  (gr_text "JLCJLCJLCJLC" (at 163 109.3 270) (layer "F.SilkS")
     (effects (font (size 1.5 1.5) (thickness 0.3)))
   )
@@
     (polygon
       (pts
-        (xy 260 137.5)
-        (xy 158.9 137.6)
+        (xy 259.996065 133.521762)
+        (xy 158.896065 133.621762)
         (xy 158.8 27.5)
         (xy 259.9 27.5)
