File: esp-merged kicad/esp-merged_v2/esp-merged_v2.kicad_sch (KiCad schematic)
At the start: 19 parts, among them J1 Conn_02x04_Male, J2 SD_Card, J3 Screw_Terminal_01x12, M1 HX711, SW1 SW_Push, SW2 SW_Push, U1 ESP32-WROOM-32, U2 SIM800L, U3 DS3231M

Commit message: a
Other:
- note removed: "todo miejsca na srubki, w tym pod koszykiem"
Changed lines of the file:
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@@
-    (effects (font (size 1.27 1.27)) (justify left bottom))
-  )
-  (text "todo miejsca na srubki, w tym pod koszykiem" (at 39.37 20.32 0)
     (effects (font (size 1.27 1.27)) (justify left bottom))
   )
