File: projekt PCB/esp-merged kicad/esp_merged_v2/esp-merged_v2.kicad_sch (KiCad schematic)
At the start: 19 parts, among them J1 Conn_02x04_Male, J2 SD_Card, J3 Screw_Terminal_01x12, M1 HX711, SW1 SW_Push, SW2 SW_Push, U1 ESP32-WROOM-32, U2 SIM800L, U3 DS3231M

Commit message: początki fixów do schematu pcb v2
Parts:
- added J? (x3): Conn_01x02_Male, symbol Connector:Conn_01x02_Male
- added R?: 75, symbol Device:R
- added R?: 36, symbol Device:R
- added R?: 10K, symbol Device:R
Connections:
- net 3.3 VCC: now also J?.1 (Pin_1)
- net GND: now also R?.1, R?.1, R?.2
- net sim reset: now reaches U2.3 (RST)
- net sim wakeUp: now reaches U2.7 (DTR)
- new net: J?.1 (Pin_1), R?.2 (x2)
- new net btnWakeUp: J?.2 (Pin_2), R?.1
- new net ledGreen: J?.2 (Pin_2)
- new net ledRed: J?.2 (Pin_2)
- no-connect marks 36 -> 34
Other:
- note added: "Budzenie ze snu"
- note added: "Sygnalizacja"
- note added: "do montażu na krawędzi płytki"
- note added: "do przycisku na zewnątrz obudowy do budzenia"
- note added: "teoretycznie 36ohm, może być 100ohm"
- note added: "teoretycznie 75ohm, może być 100ohm"
- note added: "todo"
- note added: "todo TP4056 i ładowanie (po testach wczesniejszych)"
- note removed: "todo jako antene dać wyjście odpowiednie do podłączenia PCB pod kabel i kablem do anteny"
- note removed: "todo rozważyć orientację i stronę po której będzie footprint do interfrejsu PROG, jeśli się okaże że wszystkie komponenty będą po jednej stronie to możliwe, że żeby programować płytkę będzie trzeba ją do góry nogami dać do adaptera, więc obecny footprint może musieć być na odwrót"

Commit message: maly progress pcb
Parts:
- removed F1: Fuse, Resistor_THT:R_Axial_DIN0411_L9.9mm_D3.6mm_P15.24mm_Horizontal, symbol Device:Fuse
- removed J1: Conn_02x04_Male, wlasne_footprinty:prog pins ESP32 (aka esp01) v2 (odwrocone), symbol Connector:Conn_01x08_Male
- removed SW1: SW_Push, wlasne_footprinty:wlacznik, symbol Switch:SW_Push
- removed SW2: SW_Push, wlasne_footprinty:mały button, symbol Switch:SW_Push
- removed U3: DS3231M, wlasne_footprinty:ds3231, symbol Timer_RTC:DS3231M
- added C?: 47uF, symbol Device:C_Polarized
- added F?: Fuse, Resistor_THT:R_Axial_DIN0411_L9.9mm_D3.6mm_P15.24mm_Horizontal, symbol Device:Fuse
- added J?: Conn_01x02_Female, symbol Connector:Conn_01x02_Female
- added J?: 8P8C, wlasne_footprinty:Ethernet 8p8c moje, symbol Connector:8P8C
- added SW?: SW_Push, wlasne_footprinty:wlacznik, symbol Switch:SW_Push
- added T?: tp4056, symbol wlasna_biblioteka1:tp4056
Connections:
- net 3.3 VCC: now also C?.1, J?.4
- net Battery VCC: now also F?.2
- net GND: now also C?.2, J?.3, T?.6 (Out-); no longer BT1.2 (-)
- net PROG_EN: now also J?.6
- net PROG_I0: now also J?.5
- net PROG_RX: now also J?.1
- net PROG_TX: now also J?.8
- net sim reset: now also U1.12 (IO27)
- net sim wakeUp: now also U1.16 (IO13)
- net at BT1.1 (+): now also T?.3 (Battery+)
- new net: SW?.1, T?.5 (Out+)
- new net: F?.1, SW?.2
- new net: J?.2 (Pin_2), T?.1 (Input+)
- new net: J?.1 (Pin_1), T?.2 (Input-)
- new net: BT1.2 (-), T?.4 (Battery-)
- no-connect marks 34 -> 24
Other:
- note added: "Interfejs prog"
- note added: "Zasilanie"
- note added: "konektor na zewn dla solara"
- note added: "todo chyba jeden led starczy"
- note added: "todo footprint tp4056"
- note added: "todo konieczny test, czy tp odpowiednio będzie przełączać prąd pomiędzy baterią a słabym źródłem prądu jak solar sim i esp nie mogą się resetować"
- note removed: "Wyjścia do programowania w układzie esp-01, tak aby możliwe było połączenie poprzez programator (męskie piny do góry płytki, elementem odwracanym jest adapter)"
- note removed: "Zegar czasu rzeczywistego"
- moved on the sheet: BT1, J2, J?, R?, S1

Commit message: app front adjustments
Parts:
- removed J?: Conn_01x02_Male, symbol Connector:Conn_01x02_Male
- removed R?: 36, symbol Device:R
- T?: footprint (none) -> wlasne_footprinty:tp4056
Connections:
- net ledRed: now also U1.18 (SWP/SD3)
- no-connect marks 24 -> 23
Other:
- note added: "todo connector na 2 wyjscia, z footprintem tych moich do zasilania"
- note added: "todo footprint sim800L poprawic"
- note added: "todo przetestowac czy tp4056 jest potrzebny w ogole, byc moze starczy uklad z pudelka na baterie"
- note removed: "teoretycznie 36ohm, może być 100ohm"
- note removed: "todo"
- note removed: "todo chyba jeden led starczy"
- note removed: "todo footprint tp4056"
Changed lines of the file:
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@@
   (no_connect (at 224.79 79.375))
   (no_connect (at 163.83 118.11))
-  (no_connect (at 39.37 107.315))
   (no_connect (at 139.065 54.61))
   (no_connect (at 69.85 127.635))
@@
     (stroke (width 0) (type default) (color 0 0 0 0))
   )
-  (polyline (pts (xy 233.68 44.45) (xy 233.68 64.77))
+  (polyline (pts (xy 233.045 44.45) (xy 233.045 64.77))
     (stroke (width 0) (type default) (color 0 0 0 0))
   )
@@
     (stroke (width 0) (type default) (color 0 0 0 0))
   )
-  (polyline (pts (xy 233.68 64.77) (xy 278.13 64.77))
+  (polyline (pts (xy 233.045 64.77) (xy 278.13 64.77))
     (stroke (width 0) (type default) (color 0 0 0 0))
   )
@@
     (stroke (width 0) (type default) (color 0 0 0 0))
   )
-  (polyline (pts (xy 278.13 44.45) (xy 233.68 44.45))
+  (polyline (pts (xy 278.13 44.45) (xy 233.045 44.45))
     (stroke (width 0) (type default) (color 0 0 0 0))
   )
@@
   )
   (wire (pts (xy 175.895 46.99) (xy 177.165 46.99))
-    (stroke (width 0) (type default) (color 0 0 0 0))
-  )
-  (wire (pts (xy 245.11 149.225) (xy 250.825 149.225))
     (stroke (width 0) (type default) (color 0 0 0 0))
   )
@@
     (effects (font (size 1.27 1.27)) (justify left bottom))
   )
+  (text "todo przetestowac czy tp4056 jest potrzebny w ogole, byc moze\nstarczy uklad z pudelka na baterie"
+    (at 28.575 151.765 0)
+    (effects (font (size 1.27 1.27)) (justify left bottom))
+  )
   (text "ESP MERGED V1" (at 106.68 21.59 0)
     (effects (font (size 5 5)) (justify left bottom))
@@
     (effects (font (size 1.27 1.27)) (justify left bottom))
   )
-  (text "todo" (at 233.68 147.955 0)
-    (effects (font (size 1.27 1.27)) (justify left bottom))
-  )
-  (text "todo" (at 192.405 147.955 0)
+  (text "todo footprint sim800L poprawic" (at 41.275 162.56 0)
     (effects (font (size 1.27 1.27)) (justify left bottom))
   )
@@
   )
   (text "Czujnik wstrząsów (zewnętrzny moduł)" (at 241.3 44.45 0)
-    (effects (font (size 1.27 1.27)) (justify left bottom))
-  )
-  (text "todo chyba jeden led starczy" (at 212.09 142.24 0)
     (effects (font (size 1.27 1.27)) (justify left bottom))
   )
@@
     (effects (font (size 1.27 1.27)) (justify left bottom))
   )
-  (text "do montażu na krawędzi płytki" (at 238.76 161.925 0)
-    (effects (font (size 1.27 1.27)) (justify left bottom))
-  )
   (text "do montażu na krawędzi płytki" (at 193.04 162.56 0)
     (effects (font (size 1.27 1.27)) (justify left bottom))
   )
+  (text "todo connector na 2 wyjscia, z footprintem tych moich do zasilania"
+    (at 116.84 136.525 0)
+    (effects (font (size 1.27 1.27)) (justify left bottom))
+  )
   (text "Budzenie ze snu" (at 233.045 21.59 0)
     (effects (font (size 1.27 1.27)) (justify left bottom))
@@
     (effects (font (size 1.27 1.27)) (justify left bottom))
   )
-  (text "teoretycznie 36ohm, może być 100ohm" (at 238.76 159.385 0)
-    (effects (font (size 1.27 1.27)) (justify left bottom))
-  )
   (text "Waga" (at 181.61 67.945 0)
     (effects (font (size 1.27 1.27)) (justify left bottom))
@@
     (effects (font (size 1.27 1.27)) (justify left bottom))
   )
-  (text "todo footprint tp4056\n" (at 111.76 175.26 0)
-    (effects (font (size 1.27 1.27)) (justify left bottom))
-  )
   (label "CS" (at 69.85 81.915 0)
     (effects (font (size 1.27 1.27)) (justify left bottom))
+  )
+  (label "ledRed" (at 39.37 107.315 180)
+    (effects (font (size 1.27 1.27)) (justify right bottom))
   )
   (label "sim reset" (at 69.85 117.475 0)
@@
   )
   (label "PROG_EN" (at 35.56 85.09 180)
-    (effects (font (size 1.27 1.27)) (justify right bottom))
-  )
-  (label "ledGreen" (at 245.11 149.225 180)
     (effects (font (size 1.27 1.27)) (justify right bottom))
   )
@@
     )
     (property "Datasheet" "~" (id 3) (at 212.09 151.765 0)
-      (effects (font (size 1.27 1.27)) hide)
-    )
-    (pin "1")
-    (pin "2")
-  )
-  (symbol (lib_id "Connector:Conn_01x02_Male") (at 255.905 151.765 180) (unit 1)
-    (in_bom yes) (on_board yes) (fields_autoplaced)
-    (property "Reference" "J?" (id 0) (at 257.175 149.2249 0)
-      (effects (font (size 1.27 1.27)) (justify right))
-    )
-    (property "Value" "Conn_01x02_Male" (id 1) (at 257.175 151.7649 0)
-      (effects (font (size 1.27 1.27)) (justify right))
-    )
-    (property "Footprint" "" (id 2) (at 255.905 151.765 0)
-      (effects (font (size 1.27 1.27)) hide)
-    )
-    (property "Datasheet" "~" (id 3) (at 255.905 151.765 0)
       (effects (font (size 1.27 1.27)) hide)
     )
@@
     (pin "1")
   )
-  (symbol (lib_id "power:GND") (at 243.205 151.765 270) (unit 1)
-    (in_bom yes) (on_board yes) (fields_autoplaced)
-    (property "Reference" "#PWR?" (id 0) (at 236.855 151.765 0)
-      (effects (font (size 1.27 1.27)) hide)
-    )
-    (property "Value" "GND" (id 1) (at 240.03 151.7649 90)
-      (effects (font (size 1.27 1.27)) (justify right))
-    )
-    (property "Footprint" "" (id 2) (at 243.205 151.765 0)
-      (effects (font (size 1.27 1.27)) hide)
-    )
-    (property "Datasheet" "" (id 3) (at 243.205 151.765 0)
-      (effects (font (size 1.27 1.27)) hide)
-    )
-    (pin "1")
-  )
   (symbol (lib_id "Device:Fuse") (at 170.815 151.13 90) (unit 1)
     (in_bom yes) (on_board yes) (fields_autoplaced)
@@
     (property "Reference" "T?" (id 0) (at 136.525 161.29 0))
     (property "Value" "tp4056" (id 1) (at 142.875 161.29 0))
-    (property "Footprint" "" (id 2) (at 133.985 149.86 0)
+    (property "Footprint" "wlasne_footprinty:tp4056" (id 2) (at 133.985 149.86 0)
       (effects (font (size 1.27 1.27)) hide)
     )
@@
     )
     (pin "1")
-  )
-  (symbol (lib_id "Device:R") (at 247.015 151.765 90) (unit 1)
-    (in_bom yes) (on_board yes)
-    (property "Reference" "R?" (id 0) (at 247.015 155.575 90))
-    (property "Value" "36" (id 1) (at 247.015 153.67 90))
-    (property "Footprint" "" (id 2) (at 247.015 153.543 90)
-      (effects (font (size 1.27 1.27)) hide)
-    )
-    (property "Datasheet" "~" (id 3) (at 247.015 151.765 0)
-      (effects (font (size 1.27 1.27)) hide)
-    )
-    (pin "1")
-    (pin "2")
   )
   (symbol (lib_id "Device:C_Polarized") (at 139.7 87.63 0) (unit 1)
@@
       (reference "#PWR?") (unit 1) (value "GND") (footprint "")
     )
-    (path "/222dc065-5402-4a47-b7a9-30d0ea70c561"
-      (reference "#PWR?") (unit 1) (value "GND") (footprint "")
-    )
     (path "/4f3feea6-56c2-4217-a555-54fb3b1e4fee"
       (reference "#PWR?") (unit 1) (value "GND") (footprint "")
@@
       (reference "J?") (unit 1) (value "Conn_01x02_Male") (footprint "")
     )
-    (path "/11a4c3d1-9540-481a-ae2b-6bc402432d87"
-      (reference "J?") (unit 1) (value "Conn_01x02_Male") (footprint "")
-    )
     (path "/5ed9e3cc-903d-4e9d-add0-8aecb96bb85a"
       (reference "J?") (unit 1) (value "Conn_01x02_Male") (footprint "")
@@
       (reference "R?") (unit 1) (value "75") (footprint "")
     )
-    (path "/51cd2618-7f99-4bb8-88fb-63fbdb5246ae"
-      (reference "R?") (unit 1) (value "36") (footprint "")
-    )
     (path "/e7a83459-118f-42a0-9149-222c5db4fd9b"
       (reference "R?") (unit 1) (value "10K") (footprint "")
@@
     )
     (path "/299be0ce-2c82-4e62-98f7-36efa0be3d90"
-      (reference "T?") (unit 1) (value "tp4056") (footprint "")
+      (reference "T?") (unit 1) (value "tp4056") (footprint "wlasne_footprinty:tp4056")
     )
     (path "/d61b37e6-1acd-4826-b1f1-a50ad37b0751"
